File: PCB/Design/Clock.brd (EAGLE design)
At the start: 80 x 80 mm, 83 parts, among them U1 ATMEGA644P-20AU

Commit message: connected all PWM and LEDs.
Parts:
- moved U5 53.7 mm to (67.1, 45.1), flipped to the bottom, turned to 258 degrees
- moved U9 52.8 mm to (21.7, 61.3), flipped to the bottom, turned to 138 degrees
- moved U12 51.1 mm to (65.9, 30.9), flipped to the bottom, turned to 288 degrees
- moved U10 49.5 mm to (34.7, 67.8), flipped to the bottom, turned to 168 degrees
- moved U13 40.6 mm to (18.4, 21.7), flipped to the bottom, turned to 48 degrees
- moved U6 40.0 mm to (45.2, 12.7), flipped to the bottom, turned to 348 degrees
- moved U4 34.2 mm to (12.9, 34.8), flipped to the bottom, turned to 78 degrees
- moved U7 34.2 mm to (58.3, 18.9), flipped to the bottom, turned to 318 degrees
- moved U8 33.2 mm to (30.9, 13.4), flipped to the bottom, turned to 18 degrees
- moved U11 20.2 mm to (13.5, 49.4), flipped to the bottom, turned to 108 degrees
- moved U3 20.0 mm to (61.1, 58.2), flipped to the bottom, turned to 228 degrees
Connections:
- new net DGND: U10.11, U10.M, U11.11, U11.M, U12.11, U12.M, U13.11, U13.M, U2.11, U2.M, U3.11, U3.M, U4.11, U4.M, U5.11, U5.M, U6.11, U6.M, U7.11, U7.M, U8.11, U8.M, U9.11, U9.M
- new net N$100: LED44.1, U4.15
- new net N$101: LED45.3, U4.16
- new net N$102: LED45.2, U4.17
- new net N$103: LED45.1, U4.18
- new net N$104: LED38.3, U13.9
- new net N$105: LED38.1, U13.12
- new net N$106: LED37.1, U13.8
- new net N$107: LED37.2, U13.7
- new net N$108: LED37.3, U13.6
- new net N$109: LED36.1, U13.5
- new net N$110: LED36.2, U13.4
- new net N$111: LED36.3, U13.3
- new net N$112: LED39.3, U13.13
- new net N$113: LED39.2, U13.14
- new net N$114: LED39.1, U13.15
- new net N$115: LED40.3, U13.16
- new net N$116: LED40.2, U13.17
- new net N$117: LED40.1, U13.18
- new net N$118: LED33.3, U8.9
- new net N$119: LED33.1, U8.12
- new net N$120: LED32.1, U8.8
- new net N$121: LED32.2, U8.7
- new net N$122: LED32.3, U8.6
- new net N$123: LED31.1, U8.5
- new net N$124: LED31.2, U8.4
- new net N$125: LED31.3, U8.3
- new net N$126: LED34.3, U8.13
- new net N$127: LED34.2, U8.14
- new net N$128: LED34.1, U8.15
- new net N$129: LED35.3, U8.16
- new net N$130: LED35.2, U8.17
- new net N$131: LED35.1, U8.18
- new net N$132: LED48.3, U11.9
- new net N$133: LED48.1, U11.12
- new net N$134: LED47.1, U11.8
- new net N$135: LED47.2, U11.7
- new net N$136: LED47.3, U11.6
- new net N$137: LED46.1, U11.5
- new net N$138: LED46.2, U11.4
- new net N$139: LED46.3, U11.3
- new net N$140: LED49.3, U11.13
- new net N$141: LED49.2, U11.14
- new net N$142: LED49.1, U11.15
- new net N$143: LED50.3, U11.16
- new net N$144: LED50.2, U11.17
- new net N$145: LED50.1, U11.18
- new net N$146: LED53.3, U9.9
- new net N$147: LED53.1, U9.12
- new net N$148: LED52.1, U9.8
- new net N$149: LED52.2, U9.7
- new net N$150: LED52.3, U9.6
- new net N$151: LED51.1, U9.5
- new net N$152: LED51.2, U9.4
- new net N$153: LED51.3, U9.3
- new net N$154: LED54.3, U9.13
- new net N$155: LED54.2, U9.14
- new net N$156: LED54.1, U9.15
- new net N$157: LED55.3, U9.16
- new net N$158: LED55.2, U9.17
- new net N$159: LED55.1, U9.18
- new net N$160: LED58.3, U10.9
- new net N$161: LED58.1, U10.12
- new net N$162: LED57.1, U10.8
- new net N$163: LED57.2, U10.7
- new net N$164: LED57.3, U10.6
- new net N$165: LED56.1, U10.5
- new net N$166: LED56.2, U10.4
- new net N$167: LED56.3, U10.3
- new net N$168: LED59.3, U10.13
- new net N$169: LED59.2, U10.14
- new net N$170: LED59.1, U10.15
- new net N$171: LED60.3, U10.16
- new net N$172: LED60.2, U10.17
- new net N$173: LED60.1, U10.18
- new net N$174: LED48.2, U11.10
- new net N$175: LED53.2, U9.10
- new net N$176: LED58.2, U10.10
- new net N$177: LED43.2, U4.10
- new net N$178: LED38.2, U13.10
- new net N$179: LED33.2, U8.10
- new net N$180: LED18.2, U12.10
- new net N$181: LED23.2, U7.10
- new net N$182: LED28.2, U6.10
- new net N$183: LED13.2, U5.10
- new net N$184: LED8.2, U3.10
- new net N$2: LED8.3, U3.9
- new net N$21: LED8.1, U3.12
- new net N$22: LED7.1, U3.8
- new net N$23: LED7.2, U3.7
- new net N$24: LED7.3, U3.6
- new net N$25: LED6.1, U3.5
- new net N$26: LED6.2, U3.4
- new net N$27: LED6.3, U3.3
- new net N$28: LED9.3, U3.13
- new net N$29: LED9.2, U3.14
- new net N$30: LED9.1, U3.15
- new net N$31: LED10.3, U3.16
- new net N$32: LED10.2, U3.17
- new net N$33: LED10.1, U3.18
- new net N$34: LED13.3, U5.9
- new net N$35: LED13.1, U5.12
- new net N$36: LED12.1, U5.8
- new net N$37: LED12.2, U5.7
- new net N$38: LED12.3, U5.6
- new net N$39: LED11.1, U5.5
- new net N$40: LED11.2, U5.4
- new net N$41: LED11.3, U5.3
- new net N$42: LED14.3, U5.13
- new net N$43: LED14.2, U5.14
- new net N$44: LED14.1, U5.15
- new net N$45: LED15.3, U5.16
- new net N$46: LED15.2, U5.17
- new net N$47: LED15.1, U5.18
- new net N$48: LED18.3, U12.9
- new net N$49: LED18.1, U12.12
- new net N$50: LED17.1, U12.8
- new net N$51: LED17.2, U12.7
- new net N$52: LED17.3, U12.6
- new net N$53: LED16.1, U12.5
- new net N$54: LED16.2, U12.4
- new net N$55: LED16.3, U12.3
- new net N$56: LED19.3, U12.13
- new net N$57: LED19.2, U12.14
- new net N$58: LED19.1, U12.15
- new net N$59: LED20.3, U12.16
- new net N$60: LED20.2, U12.17
- new net N$61: LED20.1, U12.18
- new net N$62: LED23.3, U7.9
- new net N$63: LED23.1, U7.12
- new net N$64: LED22.1, U7.8
- new net N$65: LED22.2, U7.7
- new net N$66: LED22.3, U7.6
- new net N$67: LED21.1, U7.5
- new net N$68: LED21.2, U7.4
- new net N$69: LED21.3, U7.3
- new net N$70: LED24.3, U7.13
- new net N$71: LED24.2, U7.14
- new net N$72: LED24.1, U7.15
- new net N$73: LED25.3, U7.16
- new net N$74: LED25.2, U7.17
- new net N$75: LED25.1, U7.18
- new net N$76: LED28.3, U6.9
- new net N$77: LED28.1, U6.12
- new net N$78: LED27.1, U6.8
- new net N$79: LED27.2, U6.7
- new net N$80: LED27.3, U6.6
- new net N$81: LED26.1, U6.5
- new net N$82: LED26.2, U6.4
- new net N$83: LED26.3, U6.3
- new net N$84: LED29.3, U6.13
- new net N$85: LED29.2, U6.14
- new net N$86: LED29.1, U6.15
- new net N$87: LED30.3, U6.16
- new net N$88: LED30.2, U6.17
- new net N$89: LED30.1, U6.18
- new net N$90: LED43.3, U4.9
- new net N$91: LED43.1, U4.12
- new net N$92: LED42.1, U4.8
- new net N$93: LED42.2, U4.7
- new net N$94: LED42.3, U4.6
- new net N$95: LED41.1, U4.5
- new net N$96: LED41.2, U4.4
- new net N$97: LED41.3, U4.3
- new net N$98: LED44.3, U4.13
- new net N$99: LED44.2, U4.14
- net GND: no longer U10.11, U10.M, U11.11, U11.M, U12.11, U12.M, U13.11, U13.M, U2.11, U2.M, U3.11, U3.M, U4.11, U4.M, U5.11, U5.M, U6.11, U6.M, U7.11, U7.M, U8.11, U8.M, U9.11, U9.M

Commit message: Probably joined with last commit..
Connections:
- removed net +5V: U1.17, U1.27, U1.38, U1.5
- removed net BLUE_CS: U1.42
- removed net GREEN_CS: U1.41
- removed net RED_CS: U1.40
- removed net SPI_CLK: U1.3
- removed net SPI_MISO: U1.2
- removed net SPI_MOSI: U1.1
- removed net VDD: U10.25, U11.25, U12.25, U13.25, U2.25, U3.25, U4.25, U5.25, U6.25, U7.25, U8.25, U9.25
- new net BANK10_OE#: U11.20
- new net BANK11_OE#: U9.20
- new net BANK12_OE#: U10.20
- new net BANK1_OE#: U2.20
- new net BANK2_OE#: U3.20
- new net BANK3_OE#: U5.20
- new net BANK4_OE#: U12.20
- new net BANK5_OE#: U7.20
- new net BANK6_OE#: U6.20
- new net BANK7_OE#: U8.20
- new net BANK8_OE#: U13.20
- new net BANK9_OE#: U4.20
- new net N$185: U6.22
- new net SCL: U10.23, U11.23, U12.23, U13.23, U2.23, U3.23, U4.23, U5.23, U6.23, U7.23, U8.23, U9.23
- new net SDA: U10.24, U11.24, U12.24, U13.24, U2.24, U3.24, U4.24, U5.24, U6.24, U7.24, U8.24, U9.24
- new net VCC: U1.17, U1.27, U1.38, U1.5, U10.25, U11.25, U12.25, U13.25, U2.25, U3.25, U4.25, U5.25, U6.25, U7.25, U8.25, U9.25
- net DGND: now also U10.22, U11.22, U12.22, U13.22, U2.22, U3.22, U4.22, U5.22, U7.22, U8.22, U9.22
