File: PCB/Design/Clock.sch (EAGLE design)
At the start: 83 parts, among them U1 ATMEGA644P-20AU

Commit message: connected all PWM and LEDs.
Connections:
- new net DGND: U10.GND, U11.GND, U12.GND, U13.GND, U2.GND, U3.GND, U4.GND, U5.GND, U6.GND, U7.GND, U8.GND, U9.GND
- new net N$100: LED44.BLUE_C, U4.PWM11
- new net N$101: LED45.RED_C, U4.PWM12
- new net N$102: LED45.GREEN_C, U4.PWM13
- new net N$103: LED45.BLUE_C, U4.PWM14
- new net N$104: LED38.RED_C, U13.PWM6
- new net N$105: LED38.BLUE_C, U13.PWM8
- new net N$106: LED37.BLUE_C, U13.PWM5
- new net N$107: LED37.GREEN_C, U13.PWM4
- new net N$108: LED37.RED_C, U13.PWM3
- new net N$109: LED36.BLUE_C, U13.PWM2
- new net N$110: LED36.GREEN_C, U13.PWM1
- new net N$111: LED36.RED_C, U13.PWM0
- new net N$112: LED39.RED_C, U13.PWM9
- new net N$113: LED39.GREEN_C, U13.PWM10
- new net N$114: LED39.BLUE_C, U13.PWM11
- new net N$115: LED40.RED_C, U13.PWM12
- new net N$116: LED40.GREEN_C, U13.PWM13
- new net N$117: LED40.BLUE_C, U13.PWM14
- new net N$118: LED33.RED_C, U8.PWM6
- new net N$119: LED33.BLUE_C, U8.PWM8
- new net N$120: LED32.BLUE_C, U8.PWM5
- new net N$121: LED32.GREEN_C, U8.PWM4
- new net N$122: LED32.RED_C, U8.PWM3
- new net N$123: LED31.BLUE_C, U8.PWM2
- new net N$124: LED31.GREEN_C, U8.PWM1
- new net N$125: LED31.RED_C, U8.PWM0
- new net N$126: LED34.RED_C, U8.PWM9
- new net N$127: LED34.GREEN_C, U8.PWM10
- new net N$128: LED34.BLUE_C, U8.PWM11
- new net N$129: LED35.RED_C, U8.PWM12
- new net N$130: LED35.GREEN_C, U8.PWM13
- new net N$131: LED35.BLUE_C, U8.PWM14
- new net N$132: LED48.RED_C, U11.PWM6
- new net N$133: LED48.BLUE_C, U11.PWM8
- new net N$134: LED47.BLUE_C, U11.PWM5
- new net N$135: LED47.GREEN_C, U11.PWM4
- new net N$136: LED47.RED_C, U11.PWM3
- new net N$137: LED46.BLUE_C, U11.PWM2
- new net N$138: LED46.GREEN_C, U11.PWM1
- new net N$139: LED46.RED_C, U11.PWM0
- new net N$140: LED49.RED_C, U11.PWM9
- new net N$141: LED49.GREEN_C, U11.PWM10
- new net N$142: LED49.BLUE_C, U11.PWM11
- new net N$143: LED50.RED_C, U11.PWM12
- new net N$144: LED50.GREEN_C, U11.PWM13
- new net N$145: LED50.BLUE_C, U11.PWM14
- new net N$146: LED53.RED_C, U9.PWM6
- new net N$147: LED53.BLUE_C, U9.PWM8
- new net N$148: LED52.BLUE_C, U9.PWM5
- new net N$149: LED52.GREEN_C, U9.PWM4
- new net N$150: LED52.RED_C, U9.PWM3
- new net N$151: LED51.BLUE_C, U9.PWM2
- new net N$152: LED51.GREEN_C, U9.PWM1
- new net N$153: LED51.RED_C, U9.PWM0
- new net N$154: LED54.RED_C, U9.PWM9
- new net N$155: LED54.GREEN_C, U9.PWM10
- new net N$156: LED54.BLUE_C, U9.PWM11
- new net N$157: LED55.RED_C, U9.PWM12
- new net N$158: LED55.GREEN_C, U9.PWM13
- new net N$159: LED55.BLUE_C, U9.PWM14
- new net N$160: LED58.RED_C, U10.PWM6
- new net N$161: LED58.BLUE_C, U10.PWM8
- new net N$162: LED57.BLUE_C, U10.PWM5
- new net N$163: LED57.GREEN_C, U10.PWM4
- new net N$164: LED57.RED_C, U10.PWM3
- new net N$165: LED56.BLUE_C, U10.PWM2
- new net N$166: LED56.GREEN_C, U10.PWM1
- new net N$167: LED56.RED_C, U10.PWM0
- new net N$168: LED59.RED_C, U10.PWM9
- new net N$169: LED59.GREEN_C, U10.PWM10
- new net N$170: LED59.BLUE_C, U10.PWM11
- new net N$171: LED60.RED_C, U10.PWM12
- new net N$172: LED60.GREEN_C, U10.PWM13
- new net N$173: LED60.BLUE_C, U10.PWM14
- new net N$174: LED48.GREEN_C, U11.PWM7
- new net N$175: LED53.GREEN_C, U9.PWM7
- new net N$176: LED58.GREEN_C, U10.PWM7
- new net N$177: LED43.GREEN_C, U4.PWM7
- new net N$178: LED38.GREEN_C, U13.PWM7
- new net N$179: LED33.GREEN_C, U8.PWM7
- new net N$180: LED18.GREEN_C, U12.PWM7
- new net N$181: LED23.GREEN_C, U7.PWM7
- new net N$182: LED28.GREEN_C, U6.PWM7
- new net N$183: LED13.GREEN_C, U5.PWM7
- new net N$184: LED8.GREEN_C, U3.PWM7
- new net N$2: LED8.RED_C, U3.PWM6
- new net N$21: LED8.BLUE_C, U3.PWM8
- new net N$22: LED7.BLUE_C, U3.PWM5
- new net N$23: LED7.GREEN_C, U3.PWM4
- new net N$24: LED7.RED_C, U3.PWM3
- new net N$25: LED6.BLUE_C, U3.PWM2
- new net N$26: LED6.GREEN_C, U3.PWM1
- new net N$27: LED6.RED_C, U3.PWM0
- new net N$28: LED9.RED_C, U3.PWM9
- new net N$29: LED9.GREEN_C, U3.PWM10
- new net N$30: LED9.BLUE_C, U3.PWM11
- new net N$31: LED10.RED_C, U3.PWM12
- new net N$32: LED10.GREEN_C, U3.PWM13
- new net N$33: LED10.BLUE_C, U3.PWM14
- new net N$34: LED13.RED_C, U5.PWM6
- new net N$35: LED13.BLUE_C, U5.PWM8
- new net N$36: LED12.BLUE_C, U5.PWM5
- new net N$37: LED12.GREEN_C, U5.PWM4
- new net N$38: LED12.RED_C, U5.PWM3
- new net N$39: LED11.BLUE_C, U5.PWM2
- new net N$40: LED11.GREEN_C, U5.PWM1
- new net N$41: LED11.RED_C, U5.PWM0
- new net N$42: LED14.RED_C, U5.PWM9
- new net N$43: LED14.GREEN_C, U5.PWM10
- new net N$44: LED14.BLUE_C, U5.PWM11
- new net N$45: LED15.RED_C, U5.PWM12
- new net N$46: LED15.GREEN_C, U5.PWM13
- new net N$47: LED15.BLUE_C, U5.PWM14
- new net N$48: LED18.RED_C, U12.PWM6
- new net N$49: LED18.BLUE_C, U12.PWM8
- new net N$50: LED17.BLUE_C, U12.PWM5
- new net N$51: LED17.GREEN_C, U12.PWM4
- new net N$52: LED17.RED_C, U12.PWM3
- new net N$53: LED16.BLUE_C, U12.PWM2
- new net N$54: LED16.GREEN_C, U12.PWM1
- new net N$55: LED16.RED_C, U12.PWM0
- new net N$56: LED19.RED_C, U12.PWM9
- new net N$57: LED19.GREEN_C, U12.PWM10
- new net N$58: LED19.BLUE_C, U12.PWM11
- new net N$59: LED20.RED_C, U12.PWM12
- new net N$60: LED20.GREEN_C, U12.PWM13
- new net N$61: LED20.BLUE_C, U12.PWM14
- new net N$62: LED23.RED_C, U7.PWM6
- new net N$63: LED23.BLUE_C, U7.PWM8
- new net N$64: LED22.BLUE_C, U7.PWM5
- new net N$65: LED22.GREEN_C, U7.PWM4
- new net N$66: LED22.RED_C, U7.PWM3
- new net N$67: LED21.BLUE_C, U7.PWM2
- new net N$68: LED21.GREEN_C, U7.PWM1
- new net N$69: LED21.RED_C, U7.PWM0
- new net N$70: LED24.RED_C, U7.PWM9
- new net N$71: LED24.GREEN_C, U7.PWM10
- new net N$72: LED24.BLUE_C, U7.PWM11
- new net N$73: LED25.RED_C, U7.PWM12
- new net N$74: LED25.GREEN_C, U7.PWM13
- new net N$75: LED25.BLUE_C, U7.PWM14
- new net N$76: LED28.RED_C, U6.PWM6
- new net N$77: LED28.BLUE_C, U6.PWM8
- new net N$78: LED27.BLUE_C, U6.PWM5
- new net N$79: LED27.GREEN_C, U6.PWM4
- new net N$80: LED27.RED_C, U6.PWM3
- new net N$81: LED26.BLUE_C, U6.PWM2
- new net N$82: LED26.GREEN_C, U6.PWM1
- new net N$83: LED26.RED_C, U6.PWM0
- new net N$84: LED29.RED_C, U6.PWM9
- new net N$85: LED29.GREEN_C, U6.PWM10
- new net N$86: LED29.BLUE_C, U6.PWM11
- new net N$87: LED30.RED_C, U6.PWM12
- new net N$88: LED30.GREEN_C, U6.PWM13
- new net N$89: LED30.BLUE_C, U6.PWM14
- new net N$90: LED43.RED_C, U4.PWM6
- new net N$91: LED43.BLUE_C, U4.PWM8
- new net N$92: LED42.BLUE_C, U4.PWM5
- new net N$93: LED42.GREEN_C, U4.PWM4
- new net N$94: LED42.RED_C, U4.PWM3
- new net N$95: LED41.BLUE_C, U4.PWM2
- new net N$96: LED41.GREEN_C, U4.PWM1
- new net N$97: LED41.RED_C, U4.PWM0
- new net N$98: LED44.RED_C, U4.PWM9
- new net N$99: LED44.GREEN_C, U4.PWM10
Other:
- moved on the sheet: LED10, LED11, LED12, LED13, LED14, LED15, LED16, LED17, LED18, LED19, LED20, LED21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

Commit message: Probably joined with last commit..
Connections:
- removed net +5V: U1.AVCC, U1.VCC, U1.VCC_2, U1.VCC_3
- removed net BLUE_CS: U1.PB2
- removed net GREEN_CS: U1.PB1
- removed net RED_CS: U1.PB0
- removed net SPI_CLK: U1.PB7
- removed net SPI_MISO: U1.PB6
- removed net SPI_MOSI: U1.PB5
- new net BANK10_OE#: U11.#OE
- new net BANK11_OE#: U9.#OE
- new net BANK12_OE#: U10.#OE
- new net BANK1_OE#: U2.#OE
- new net BANK2_OE#: U3.#OE
- new net BANK3_OE#: U5.#OE
- new net BANK4_OE#: U12.#OE
- new net BANK5_OE#: U7.#OE
- new net BANK6_OE#: U6.#OE
- new net BANK7_OE#: U8.#OE
- new net BANK8_OE#: U13.#OE
- new net BANK9_OE#: U4.#OE
- new net N$185: U6.EXTCLK
- new net SCL: U10.SCL, U11.SCL, U12.SCL, U13.SCL, U2.SCL, U3.SCL, U4.SCL, U5.SCL, U6.SCL, U7.SCL, U8.SCL, U9.SCL
- new net SDA: U10.SDA, U11.SDA, U12.SDA, U13.SDA, U2.SDA, U3.SDA, U4.SDA, U5.SDA, U6.SDA, U7.SDA, U8.SDA, U9.SDA
- new net VCC: U1.AVCC, U1.VCC, U1.VCC_2, U1.VCC_3, U10.VDD, U11.VDD, U12.VDD, U13.VDD, U2.VDD, U3.VDD, U4.VDD, U5.VDD, U6.VDD, U7.VDD, U8.VDD, U9.VDD
- net DGND: now also U10.EXTCLK, U11.EXTCLK, U12.EXTCLK, U13.EXTCLK, U2.EXTCLK, U3.EXTCLK, U4.EXTCLK, U5.EXTCLK, U7.EXTCLK, U8.EXTCLK, U9.EXTCLK
