File: Schematics/BPF.sch (KiCad schematic (older format))
At the start: 23 parts, among them U1 LM324

Commit message: LEDs are placed!
Worked out how to script KiCAD to do it too. Winner winner, time for a chicken dinner
Parts:
- renumbered C201 to C7, C7 to C8, C8 to C9, U1 to U20
Changed lines of the file:
@@
 $EndComp
 $Comp
-L C C8
+L C C9
 U 1 1 54A96B40
 P 8550 3900
-F 0 "C8" H 8550 4000 40  0000 L CNN
+F 0 "C9" H 8550 4000 40  0000 L CNN
 F 1 "100n" H 8556 3815 40  0000 L CNN
 F 2 "Capacitors_SMD:C_0603" H 8588 3750 30  0001 C CNN
@@
 $EndComp
 $Comp
-L C C7
+L C C8
 U 1 1 54A96B46
 P 8000 5050
-F 0 "C7" H 8000 5150 40  0000 L CNN
+F 0 "C8" H 8000 5150 40  0000 L CNN
 F 1 "100n" H 8006 4965 40  0000 L CNN
 F 2 "Capacitors_SMD:C_0603" H 8038 4900 30  0001 C CNN
@@
 V_com
 $Comp
-L LM324 U1
+L LM324 U20
 U 1 1 54A9C436
 P 3550 5150
-F 0 "U1" H 3600 5350 60  0000 C CNN
+F 0 "U20" H 3600 5350 60  0000 C CNN
 F 1 "LM324" H 3700 4950 50  0000 C CNN
 F 2 "SMD_Packages:TSSOP-14" H 3550 5150 60  0001 C CNN
@@
 $EndComp
 $Comp
-L LM324 U1
+L LM324 U20
 U 3 1 54A9C501
 P 6250 5050
-F 0 "U1" H 6300 5250 60  0000 C CNN
+F 0 "U20" H 6300 5250 60  0000 C CNN
 F 1 "LM324" H 6400 4850 50  0000 C CNN
 F 2 "SMD_Packages:TSSOP-14" H 6250 5050 60  0001 C CNN
@@
 $EndComp
 $Comp
-L LM324 U1
+L LM324 U20
 U 4 1 54A9C5CA
 P 9000 4950
-F 0 "U1" H 9050 5150 60  0000 C CNN
+F 0 "U20" H 9050 5150 60  0000 C CNN
 F 1 "LM324" H 9150 4750 50  0000 C CNN
 F 2 "SMD_Packages:TSSOP-14" H 9000 4950 60  0001 C CNN
@@
 $EndComp
 $Comp
-L LM324 U1
+L LM324 U20
 U 2 1 54A9C6AF
 P 5000 2600
-F 0 "U1" H 5050 2800 60  0000 C CNN
+F 0 "U20" H 5050 2800 60  0000 C CNN
 F 1 "LM324" H 5150 2400 50  0000 C CNN
 F 2 "SMD_Packages:TSSOP-14" H 5000 2600 60  0001 C CNN
@@
 Gain of amplifier = 100. \nFc of BPF = 60kHz\nOverall gain at 60kHz = 29dB
 $Comp
-L C C201
+L C C7
 U 1 1 54B27AC9
 P 7400 2250
-F 0 "C201" H 7400 2350 40  0000 L CNN
+F 0 "C7" H 7400 2350 40  0000 L CNN
 F 1 "1u" H 7406 2165 40  0000 L CNN
 F 2 "Capacitors_SMD:C_0603" H 7438 2100 30  0001 C CNN

Commit message: Updated schematics
Parts:
- R11: footprint Resistors_SMD:R_0402 -> Resistors_SMD:R_0603
- U20: footprint SMD_Packages:TSSOP-14 -> Housings_SOIC:SOIC-14_3.9x8.7mm_Pitch1.27mm
Changed lines of the file:
@@
 LIBS:pca9685
 LIBS:avr_jtag_header
+LIBS:linear-technology
 LIBS:Root-cache
 EELAYER 25 0
@@
 $EndComp
 $Comp
-L GND #PWR02
+L GND #PWR03
 U 1 1 54A96405
 P 3450 5650
-F 0 "#PWR02" H 3450 5400 60  0001 C CNN
+F 0 "#PWR03" H 3450 5400 60  0001 C CNN
 F 1 "GND" H 3450 5500 60  0000 C CNN
 F 2 "" H 3450 5650 60  0000 C CNN
@@
 RF_in
 $Comp
-L VPP #PWR03
+L VPP #PWR04
 U 1 1 54A96533
 P 3450 4700
-F 0 "#PWR03" H 3450 4550 60  0001 C CNN
+F 0 "#PWR04" H 3450 4550 60  0001 C CNN
 F 1 "VPP" H 3450 4850 60  0000 C CNN
 F 2 "" H 3450 4700 60  0000 C CNN
@@
 F 0 "R11" V 8630 4200 40  0000 C CNN
 F 1 "56k" V 8557 4201 40  0000 C CNN
-F 2 "Resistors_SMD:R_0402" V 8480 4200 30  0001 C CNN
+F 2 "Resistors_SMD:R_0603" V 8480 4200 30  0001 C CNN
 F 3 "" H 8550 4200 30  0000 C CNN
 	1    8550 4200
@@
 $EndComp
 $Comp
-L GND #PWR04
+L GND #PWR05
 U 1 1 54A96B5F
 P 8900 5450
-F 0 "#PWR04" H 8900 5200 60  0001 C CNN
+F 0 "#PWR05" H 8900 5200 60  0001 C CNN
 F 1 "GND" H 8900 5300 60  0000 C CNN
 F 2 "" H 8900 5450 60  0000 C CNN
@@
 $EndComp
 $Comp
-L VPP #PWR05
+L VPP #PWR06
 U 1 1 54A96B66
 P 8900 4500
-F 0 "#PWR05" H 8900 4350 60  0001 C CNN
+F 0 "#PWR06" H 8900 4350 60  0001 C CNN
 F 1 "VPP" H 8900 4650 60  0000 C CNN
 F 2 "" H 8900 4500 60  0000 C CNN
@@
 $EndComp
 $Comp
-L GND #PWR06
+L GND #PWR07
 U 1 1 54A96E24
 P 6150 5550
-F 0 "#PWR06" H 6150 5300 60  0001 C CNN
+F 0 "#PWR07" H 6150 5300 60  0001 C CNN
 F 1 "GND" H 6150 5400 60  0000 C CNN
 F 2 "" H 6150 5550 60  0000 C CNN
@@
 $EndComp
 $Comp
-L VPP #PWR07
+L VPP #PWR08
 U 1 1 54A96E2B
 P 6150 4600
-F 0 "#PWR07" H 6150 4450 60  0001 C CNN
+F 0 "#PWR08" H 6150 4450 60  0001 C CNN
 F 1 "VPP" H 6150 4750 60  0000 C CNN
 F 2 "" H 6150 4600 60  0000 C CNN
@@
 $EndComp
 $Comp
-L GND #PWR08
+L GND #PWR09
 U 1 1 54A99684
 P 3000 3350
-F 0 "#PWR08" H 3000 3100 60  0001 C CNN
+F 0 "#PWR09" H 3000 3100 60  0001 C CNN
 F 1 "GND" H 3000 3200 60  0000 C CNN
 F 2 "" H 3000 3350 60  0000 C CNN
@@
 $EndComp
 $Comp
-L VPP #PWR09
+L VPP #PWR010
 U 1 1 54A9A799
 P 8950 1750
-F 0 "#PWR09" H 8950 1600 60  0001 C CNN
+F 0 "#PWR010" H 8950 1600 60  0001 C CNN
 F 1 "VPP" H 8950 1900 60  0000 C CNN
 F 2 "" H 8950 1750 60  0000 C CNN
@@
 $EndComp
 $Comp
-L GND #PWR010
+L GND #PWR011
 U 1 1 54A9AB3A
 P 8950 3050
-F 0 "#PWR010" H 8950 2800 60  0001 C CNN
+F 0 "#PWR011" H 8950 2800 60  0001 C CNN
 F 1 "GND" H 8950 2900 60  0000 C CNN
 F 2 "" H 8950 3050 60  0000 C CNN
@@
 F 0 "U20" H 3600 5350 60  0000 C CNN
 F 1 "LM324" H 3700 4950 50  0000 C CNN
-F 2 "SMD_Packages:TSSOP-14" H 3550 5150 60  0001 C CNN
+F 2 "Housings_SOIC:SOIC-14_3.9x8.7mm_Pitch1.27mm" H 3550 5150 60  0001 C CNN
 F 3 "" H 3550 5150 60  0000 C CNN
 	1    3550 5150
@@
 F 0 "U20" H 6300 5250 60  0000 C CNN
 F 1 "LM324" H 6400 4850 50  0000 C CNN
-F 2 "SMD_Packages:TSSOP-14" H 6250 5050 60  0001 C CNN
+F 2 "Housings_SOIC:SOIC-14_3.9x8.7mm_Pitch1.27mm" H 6250 5050 60  0001 C CNN
 F 3 "" H 6250 5050 60  0000 C CNN
 	3    6250 5050
@@
 F 0 "U20" H 9050 5150 60  0000 C CNN
 F 1 "LM324" H 9150 4750 50  0000 C CNN
-F 2 "SMD_Packages:TSSOP-14" H 9000 4950 60  0001 C CNN
+F 2 "Housings_SOIC:SOIC-14_3.9x8.7mm_Pitch1.27mm" H 9000 4950 60  0001 C CNN
 F 3 "" H 9000 4950 60  0000 C CNN
 	4    9000 4950
@@
 F 0 "U20" H 5050 2800 60  0000 C CNN
 F 1 "LM324" H 5150 2400 50  0000 C CNN
-F 2 "SMD_Packages:TSSOP-14" H 5000 2600 60  0001 C CNN
+F 2 "Housings_SOIC:SOIC-14_3.9x8.7mm_Pitch1.27mm" H 5000 2600 60  0001 C CNN
 F 3 "" H 5000 2600 60  0000 C CNN
 	2    5000 2600
@@
 RF_in
 $Comp
-L GND #PWR011
+L GND #PWR012
 U 1 1 54A9FE65
 P 4900 3150
-F 0 "#PWR011" H 4900 2900 60  0001 C CNN
+F 0 "#PWR012" H 4900 2900 60  0001 C CNN
 F 1 "GND" H 4900 3000 60  0000 C CNN
 F 2 "" H 4900 3150 60  0000 C CNN
@@
 $EndComp
 $Comp
-L VPP #PWR012
+L VPP #PWR013
 U 1 1 54A9FE84
 P 4900 2100
-F 0 "#PWR012" H 4900 1950 60  0001 C CNN
+F 0 "#PWR013" H 4900 1950 60  0001 C CNN
 F 1 "VPP" H 4900 2250 60  0000 C CNN
 F 2 "" H 4900 2100 60  0000 C CNN
@@
 $EndComp
 $Comp
-L GND #PWR013
+L GND #PWR014
 U 1 1 54ADB002
 P 4400 3150
-F 0 "#PWR013" H 4400 2900 60  0001 C CNN
+F 0 "#PWR014" H 4400 2900 60  0001 C CNN
 F 1 "GND" H 4400 3000 60  0000 C CNN
 F 2 "" H 4400 3150 60  0000 C CNN
@@
 	4900 3150 4900 3000
 $Comp
-L VPP #PWR014
+L VPP #PWR015
 U 1 1 54ADC9C7
 P 3550 2050
-F 0 "#PWR014" H 3550 1900 60  0001 C CNN
+F 0 "#PWR015" H 3550 1900 60  0001 C CNN
 F 1 "VPP" H 3550 2200 60  0000 C CNN
 F 2 "" H 3550 2050 60  0000 C CNN
@@
 	3550 2150 3550 2050
 $Comp
-L GND #PWR015
+L GND #PWR016
 U 1 1 54ADCA56
 P 3600 3350
-F 0 "#PWR015" H 3600 3100 60  0001 C CNN
+F 0 "#PWR016" H 3600 3100 60  0001 C CNN
 F 1 "GND" H 3600 3200 60  0000 C CNN
 F 2 "" H 3600 3350 60  0000 C CNN
@@
 $EndComp
 $Comp
-L VPP #PWR016
+L VPP #PWR017
 U 1 1 54B27B93
 P 7400 2000
-F 0 "#PWR016" H 7400 1850 60  0001 C CNN
+F 0 "#PWR017" H 7400 1850 60  0001 C CNN
 F 1 "VPP" H 7400 2150 60  0000 C CNN
 F 2 "" H 7400 2000 60  0000 C CNN
@@
 $EndComp
 $Comp
-L GND #PWR017
+L GND #PWR018
 U 1 1 54B27BB8
 P 7400 2500
-F 0 "#PWR017" H 7400 2250 60  0001 C CNN
+F 0 "#PWR018" H 7400 2250 60  0001 C CNN
 F 1 "GND" H 7400 2350 60  0000 C CNN
 F 2 "" H 7400 2500 60  0000 C CNN
