File: Schematics/Display_Sub.sch (KiCad schematic (older format))
At the start: 8 parts, among them U501 PCA9685

Commit message: LEDs are placed!
Worked out how to script KiCAD to do it too. Winner winner, time for a chicken dinner
Parts:
- C21: renamed from C901; footprint (none) -> Capacitors_SMD:C_0603
- LED11: renamed from D501; footprint (none) -> rgb:rgbled1
- LED12: renamed from D502; footprint (none) -> rgb:rgbled1
- LED13: renamed from D503; footprint (none) -> rgb:rgbled1
- LED14: renamed from D504; footprint (none) -> rgb:rgbled1
- LED15: renamed from D505; footprint (none) -> rgb:rgbled1
- R19: renamed from R901; footprint (none) -> Resistors_SMD:R_0603
- renumbered U501 to U3

Commit message: Changed lots
Finalised the Inductor. Closes #5
Changed USB Connector. Closes #4
Added four switches for a simple interface. Closes #7
Added a power jack. Closes #3
Found RTC Oscillator. Closes #1.
Added part numbers to all major components. Closes #2
Parts:
- LED11: Part (none) -> ASMT-YTD7-0AA02; Supplier (none) -> Farnell
- U3: footprint Housings_DFN_QFN:QFN-28-1EP_6x6mm_Pitch0.65mm -> Housings_SSOP:TSSOP-28_4.4x9.7mm_Pitch0.65mm
Connections:
- net GND: now also U3.14 (VSS)

Commit message: Completed layout of 10cm board. Fixes #8
Changed lines of the file:
@@
 LIBS:pca9685
 LIBS:avr_jtag_header
-LIBS:linear-technology
 LIBS:Root-cache
 EELAYER 25 0
@@
 $Descr A4 11693 8268
 encoding utf-8
-Sheet 9 16
+Sheet 8 16
 Title ""
 Date ""
@@
 AR Path="/54B11834/54B2952B/54B11E68" Ref="U6"  Part="1"
 AR Path="/54B11834/54B29534/54B11E68" Ref="U12"  Part="1"
-F 0 "U7" H 4700 4050 60  0000 C CNN
+F 0 "U1" H 4700 4050 60  0000 C CNN
 F 1 "PCA9685" H 5350 4050 60  0000 C CNN
 F 2 "Housings_SSOP:TSSOP-28_4.4x9.7mm_Pitch0.65mm" H 5050 3150 60  0001 C CNN
@@
 AR Path="/54B11834/54B2952B/54B11EE3" Ref="#PWR0107"  Part="1"
 AR Path="/54B11834/54B29534/54B11EE3" Ref="#PWR0113"  Part="1"
-F 0 "#PWR0113" H 5050 4050 60  0001 C CNN
+F 0 "#PWR071" H 5050 4050 60  0001 C CNN
 F 1 "GND" H 5050 4150 60  0000 C CNN
 F 2 "" H 5050 4300 60  0000 C CNN
@@
 AR Path="/54B11834/54B2952B/54B11EF7" Ref="#PWR0108"  Part="1"
 AR Path="/54B11834/54B29534/54B11EF7" Ref="#PWR0114"  Part="1"
-F 0 "#PWR0114" H 5050 1250 60  0001 C CNN
+F 0 "#PWR072" H 5050 1250 60  0001 C CNN
 F 1 "VPP" H 5050 1550 60  0000 C CNN
 F 2 "" H 5050 1400 60  0000 C CNN
@@
 AR Path="/54B11834/54B2952B/54B11FAE" Ref="#PWR0109"  Part="1"
 AR Path="/54B11834/54B29534/54B11FAE" Ref="#PWR0115"  Part="1"
-F 0 "#PWR0115" H 4400 3350 60  0001 C CNN
+F 0 "#PWR073" H 4400 3350 60  0001 C CNN
 F 1 "GND" H 4400 3450 60  0000 C CNN
 F 2 "" H 4400 3600 60  0000 C CNN
@@
 AR Path="/54B11834/54B2952B/54B16870" Ref="LED26"  Part="1"
 AR Path="/54B11834/54B29534/54B16870" Ref="LED56"  Part="1"
-F 0 "LED31" H 6800 1850 50  0000 C CNN
+F 0 "LED1" H 6800 1850 50  0000 C CNN
 F 1 "LED_RGB" H 6750 1250 50  0000 C CNN
 F 2 "rgb:rgbled1" H 7100 1500 60  0001 C CNN
@@
 AR Path="/54B11834/54B2952B/54B16AF6" Ref="LED27"  Part="1"
 AR Path="/54B11834/54B29534/54B16AF6" Ref="LED57"  Part="1"
-F 0 "LED32" H 6800 2650 50  0000 C CNN
+F 0 "LED2" H 6800 2650 50  0000 C CNN
 F 1 "LED_RGB" H 6750 2050 50  0000 C CNN
 F 2 "rgb:rgbled1" H 7100 2300 60  0001 C CNN
@@
 AR Path="/54B11834/54B2952B/54B16B3B" Ref="LED28"  Part="1"
 AR Path="/54B11834/54B29534/54B16B3B" Ref="LED58"  Part="1"
-F 0 "LED33" H 6800 3400 50  0000 C CNN
+F 0 "LED3" H 6800 3400 50  0000 C CNN
 F 1 "LED_RGB" H 6750 2800 50  0000 C CNN
 F 2 "rgb:rgbled1" H 7100 3050 60  0001 C CNN
@@
 AR Path="/54B11834/54B2952B/54B16C15" Ref="LED29"  Part="1"
 AR Path="/54B11834/54B29534/54B16C15" Ref="LED59"  Part="1"
-F 0 "LED34" H 6800 4150 50  0000 C CNN
+F 0 "LED4" H 6800 4150 50  0000 C CNN
 F 1 "LED_RGB" H 6750 3550 50  0000 C CNN
 F 2 "rgb:rgbled1" H 7100 3800 60  0001 C CNN
@@
 AR Path="/54B11834/54B2952B/54B16C50" Ref="LED30"  Part="1"
 AR Path="/54B11834/54B29534/54B16C50" Ref="LED60"  Part="1"
-F 0 "LED35" H 6800 4900 50  0000 C CNN
+F 0 "LED5" H 6800 4900 50  0000 C CNN
 F 1 "LED_RGB" H 6750 4300 50  0000 C CNN
 F 2 "rgb:rgbled1" H 7100 4550 60  0001 C CNN
@@
 AR Path="/54B11834/54B2952B/54B17FD7" Ref="#PWR0110"  Part="1"
 AR Path="/54B11834/54B29534/54B17FD7" Ref="#PWR0116"  Part="1"
-F 0 "#PWR0116" H 7750 1000 60  0001 C CNN
+F 0 "#PWR074" H 7750 1000 60  0001 C CNN
 F 1 "VPP" H 7750 1300 60  0000 C CNN
 F 2 "" H 7750 1150 60  0000 C CNN
@@
 AR Path="/54B11834/54B2952B/54B18339" Ref="#PWR0111"  Part="1"
 AR Path="/54B11834/54B29534/54B18339" Ref="#PWR0117"  Part="1"
-F 0 "#PWR0117" H 3550 2600 60  0001 C CNN
+F 0 "#PWR075" H 3550 2600 60  0001 C CNN
 F 1 "VPP" H 3550 2900 60  0000 C CNN
 F 2 "" H 3550 2750 60  0000 C CNN
@@
 AR Path="/54B11834/54B2952B/54B2B528" Ref="C31"  Part="1"
 AR Path="/54B11834/54B29534/54B2B528" Ref="C32"  Part="1"
-F 0 "C26" H 4750 1850 40  0000 L CNN
+F 0 "C25" H 4750 1850 40  0000 L CNN
 F 1 "C" H 4756 1665 40  0000 L CNN
 F 2 "Capacitors_SMD:C_0603" H 4788 1600 30  0001 C CNN
@@
 AR Path="/54B11834/54B2952B/54B2B708" Ref="R29"  Part="1"
 AR Path="/54B11834/54B29534/54B2B708" Ref="R30"  Part="1"
-F 0 "R24" V 3680 3100 40  0000 C CNN
+F 0 "R23" V 3680 3100 40  0000 C CNN
 F 1 "10k" V 3607 3101 40  0000 C CNN
 F 2 "Resistors_SMD:R_0603" V 3530 3100 30  0001 C CNN
@@
 AR Path="/54B11834/54B2952B/54B2B9DA" Ref="#PWR0112"  Part="1"
 AR Path="/54B11834/54B29534/54B2B9DA" Ref="#PWR0118"  Part="1"
-F 0 "#PWR0118" H 4750 1750 60  0001 C CNN
+F 0 "#PWR076" H 4750 1750 60  0001 C CNN
 F 1 "GND" H 4750 1850 60  0000 C CNN
 F 2 "" H 4750 2000 60  0000 C CNN
