File: Schematics/Display_Sub.sch (KiCad schematic (older format))
At the start: 8 parts, among them U3 PCA9685

Commit message: Started Redesign.
Parts:
- removed LED11, LED12, LED13, LED14, LED15: LED_RGB, rgb:rgbled1, symbol LED_RGB
- added P801, P802, P803, P804, P805: CONN_01X04, Socket_Strips:Socket_Strip_Straight_2x02, symbol CONN_01X04
Connections:
- wire segments 79 -> 65

Commit message: Split design into two modules
Parts:
- removed U3: PCA9685, Housings_SSOP:TSSOP-28_4.4x9.7mm_Pitch0.65mm, symbol PCA9685
- added C101, C102: C, Capacitors_SMD:C_0603, symbol C
- added P6: CONN_01X06, JST-SH:JST-BM-06B-SRSS-TB, symbol CONN_01X06
- added R1, R2, R3, R4, R5, R6, R7, R8: 0R, Resistors_SMD:R_0603, symbol R
- added R10, R11: 10k, Resistors_SMD:R_0603, symbol R
- added U1: PCA9685, Housings_SOIC:SOIC-28_7.5x17.9mm_Pitch1.27mm, symbol PCA9685
- P801, P802, P803, P804, P805: footprint Socket_Strips:Socket_Strip_Straight_2x02 -> JST-SH:JST-BM-04B-SRSS-TB
Connections:
- wire segments 65 -> 103
Other:
- moved on the sheet: C1, R9
