File: Schematics/Root.sch (KiCad schematic (older format))
At the start: 13 parts, among them CON2 BARREL_JACK, P1 CONN_01X06, P10 CONN_01X06, P11 CONN_01X06, P12 CONN_01X06, P2 CONN_01X06, P3 CONN_01X06, P4 CONN_01X06, P5 CONN_01X06, P6 CONN_01X06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

Commit message: Sorted silkscreen out and panelized design.
Parts:
- P1, P10, P11, P12, P2, P3, P4, P5, P6, P7, P8, P9: footprint (none) -> JST-SH:JST-BM-06B-SRSS-TB
Changed lines of the file:
@@
 LIBS:contrib
 LIBS:valves
+LIBS:JST-SH
 LIBS:pca9685
-LIBS:avr_jtag_header
-LIBS:Root-cache
 EELAYER 25 0
 EELAYER END
@@
 $EndSheet
 $Comp
-L VPP #PWR11
+L VPP #PWR01
 U 1 1 54BAF809
 P 4150 3250
-F 0 "#PWR11" H 4150 3100 60  0001 C CNN
+F 0 "#PWR01" H 4150 3100 60  0001 C CNN
 F 1 "VPP" H 4150 3400 60  0000 C CNN
 F 2 "" H 4150 3250 60  0000 C CNN
@@
 	4150 3300 4150 3250
 $Comp
-L GND #PWR14
+L GND #PWR02
 U 1 1 54C94A98
 P 2550 3600
-F 0 "#PWR14" H 2550 3350 60  0001 C CNN
+F 0 "#PWR02" H 2550 3350 60  0001 C CNN
 F 1 "GND" H 2550 3450 60  0000 C CNN
 F 2 "" H 2550 3600 60  0000 C CNN
@@
 F 0 "P7" H 10400 1650 50  0000 C CNN
 F 1 "CONN_01X06" V 10500 1300 50  0000 C CNN
-F 2 "" H 10400 1300 60  0000 C CNN
+F 2 "JST-SH:JST-BM-06B-SRSS-TB" H 10400 1300 60  0001 C CNN
 F 3 "" H 10400 1300 60  0000 C CNN
 	1    10400 1300
@@
 	9800 1450 10200 1450
 $Comp
-L VPP #PWR2
+L VPP #PWR03
 U 1 1 551078A3
 P 9900 1000
-F 0 "#PWR2" H 9900 850 60  0001 C CNN
+F 0 "#PWR03" H 9900 850 60  0001 C CNN
 F 1 "VPP" H 9900 1150 60  0000 C CNN
 F 2 "" H 9900 1000 60  0000 C CNN
@@
 $EndComp
 $Comp
-L GND #PWR4
+L GND #PWR04
 U 1 1 551078C1
 P 10150 1600
-F 0 "#PWR4" H 10150 1350 60  0001 C CNN
+F 0 "#PWR04" H 10150 1350 60  0001 C CNN
 F 1 "GND" H 10150 1450 60  0000 C CNN
 F 2 "" H 10150 1600 60  0000 C CNN
@@
 F 0 "P8" H 10400 2550 50  0000 C CNN
 F 1 "CONN_01X06" V 10500 2200 50  0000 C CNN
-F 2 "" H 10400 2200 60  0000 C CNN
+F 2 "JST-SH:JST-BM-06B-SRSS-TB" H 10400 2200 60  0001 C CNN
 F 3 "" H 10400 2200 60  0000 C CNN
 	1    10400 2200
@@
 	9800 2350 10200 2350
 $Comp
-L VPP #PWR6
+L VPP #PWR05
 U 1 1 551091F0
 P 9900 1900
-F 0 "#PWR6" H 9900 1750 60  0001 C CNN
+F 0 "#PWR05" H 9900 1750 60  0001 C CNN
 F 1 "VPP" H 9900 2050 60  0000 C CNN
 F 2 "" H 9900 1900 60  0000 C CNN
@@
 $EndComp
 $Comp
-L GND #PWR8
+L GND #PWR06
 U 1 1 551091F6
 P 10150 2500
-F 0 "#PWR8" H 10150 2250 60  0001 C CNN
+F 0 "#PWR06" H 10150 2250 60  0001 C CNN
 F 1 "GND" H 10150 2350 60  0000 C CNN
 F 2 "" H 10150 2500 60  0000 C CNN
@@
 F 0 "P9" H 10400 3450 50  0000 C CNN
 F 1 "CONN_01X06" V 10500 3100 50  0000 C CNN
-F 2 "" H 10400 3100 60  0000 C CNN
+F 2 "JST-SH:JST-BM-06B-SRSS-TB" H 10400 3100 60  0001 C CNN
 F 3 "" H 10400 3100 60  0000 C CNN
 	1    10400 3100
@@
 	9800 3250 10200 3250
 $Comp
-L VPP #PWR10
+L VPP #PWR07
 U 1 1 551092A8
 P 9900 2800
-F 0 "#PWR10" H 9900 2650 60  0001 C CNN
+F 0 "#PWR07" H 9900 2650 60  0001 C CNN
 F 1 "VPP" H 9900 2950 60  0000 C CNN
 F 2 "" H 9900 2800 60  0000 C CNN
@@
 $EndComp
 $Comp
-L GND #PWR13
+L GND #PWR08
 U 1 1 551092AE
 P 10150 3400
-F 0 "#PWR13" H 10150 3150 60  0001 C CNN
+F 0 "#PWR08" H 10150 3150 60  0001 C CNN
 F 1 "GND" H 10150 3250 60  0000 C CNN
 F 2 "" H 10150 3400 60  0000 C CNN
@@
 F 0 "P10" H 10400 4350 50  0000 C CNN
 F 1 "CONN_01X06" V 10500 4000 50  0000 C CNN
-F 2 "" H 10400 4000 60  0000 C CNN
+F 2 "JST-SH:JST-BM-06B-SRSS-TB" H 10400 4000 60  0001 C CNN
 F 3 "" H 10400 4000 60  0000 C CNN
 	1    10400 4000
@@
 	9800 4150 10200 4150
 $Comp
-L VPP #PWR16
+L VPP #PWR09
 U 1 1 551092C6
 P 9900 3700
-F 0 "#PWR16" H 9900 3550 60  0001 C CNN
+F 0 "#PWR09" H 9900 3550 60  0001 C CNN
 F 1 "VPP" H 9900 3850 60  0000 C CNN
 F 2 "" H 9900 3700 60  0000 C CNN
@@
 $EndComp
 $Comp
-L GND #PWR18
+L GND #PWR010
 U 1 1 551092CC
 P 10150 4300
-F 0 "#PWR18" H 10150 4050 60  0001 C CNN
+F 0 "#PWR010" H 10150 4050 60  0001 C CNN
 F 1 "GND" H 10150 4150 60  0000 C CNN
 F 2 "" H 10150 4300 60  0000 C CNN
@@
 F 0 "P11" H 10400 5250 50  0000 C CNN
 F 1 "CONN_01X06" V 10500 4900 50  0000 C CNN
-F 2 "" H 10400 4900 60  0000 C CNN
+F 2 "JST-SH:JST-BM-06B-SRSS-TB" H 10400 4900 60  0001 C CNN
 F 3 "" H 10400 4900 60  0000 C CNN
 	1    10400 4900
@@
 	9800 5050 10200 5050
 $Comp
-L VPP #PWR20
+L VPP #PWR011
 U 1 1 551096E0
 P 9900 4600
-F 0 "#PWR20" H 9900 4450 60  0001 C CNN
+F 0 "#PWR011" H 9900 4450 60  0001 C CNN
 F 1 "VPP" H 9900 4750 60  0000 C CNN
 F 2 "" H 9900 4600 60  0000 C CNN
@@
 $EndComp
 $Comp
-L GND #PWR22
+L GND #PWR012
 U 1 1 551096E6
 P 10150 5200
-F 0 "#PWR22" H 10150 4950 60  0001 C CNN
+F 0 "#PWR012" H 10150 4950 60  0001 C CNN
 F 1 "GND" H 10150 5050 60  0000 C CNN
 F 2 "" H 10150 5200 60  0000 C CNN
@@
 F 0 "P12" H 10400 6150 50  0000 C CNN
 F 1 "CONN_01X06" V 10500 5800 50  0000 C CNN
-F 2 "" H 10400 5800 60  0000 C CNN
+F 2 "JST-SH:JST-BM-06B-SRSS-TB" H 10400 5800 60  0001 C CNN
 F 3 "" H 10400 5800 60  0000 C CNN
 	1    10400 5800
@@
 	9800 5950 10200 5950
 $Comp
-L VPP #PWR24
+L VPP #PWR013
 U 1 1 551096FE
 P 9900 5500
-F 0 "#PWR24" H 9900 5350 60  0001 C CNN
+F 0 "#PWR013" H 9900 5350 60  0001 C CNN
 F 1 "VPP" H 9900 5650 60  0000 C CNN
 F 2 "" H 9900 5500 60  0000 C CNN
@@
 $EndComp
 $Comp
-L GND #PWR26
+L GND #PWR014
 U 1 1 55109704
 P 10150 6100
-F 0 "#PWR26" H 10150 5850 60  0001 C CNN
+F 0 "#PWR014" H 10150 5850 60  0001 C CNN
 F 1 "GND" H 10150 5950 60  0000 C CNN
 F 2 "" H 10150 6100 60  0000 C CNN
@@
 F 0 "P1" H 8350 1600 50  0000 C CNN
 F 1 "CONN_01X06" V 8450 1250 50  0000 C CNN
-F 2 "" H 8350 1250 60  0000 C CNN
+F 2 "JST-SH:JST-BM-06B-SRSS-TB" H 8350 1250 60  0001 C CNN
 F 3 "" H 8350 1250 60  0000 C CNN
 	1    8350 1250
@@
 	7750 1400 8150 1400
 $Comp
-L VPP #PWR1
+L VPP #PWR015
 U 1 1 55109FFC
 P 7850 950
-F 0 "#PWR1" H 7850 800 60  0001 C CNN
+F 0 "#PWR015" H 7850 800 60  0001 C CNN
 F 1 "VPP" H 7850 1100 60  0000 C CNN
 F 2 "" H 7850 950 60  0000 C CNN
@@
 $EndComp
 $Comp
-L GND #PWR3
+L GND #PWR016
 U 1 1 5510A002
 P 8100 1550
-F 0 "#PWR3" H 8100 1300 60  0001 C CNN
+F 0 "#PWR016" H 8100 1300 60  0001 C CNN
 F 1 "GND" H 8100 1400 60  0000 C CNN
 F 2 "" H 8100 1550 60  0000 C CNN
@@
 F 0 "P2" H 8350 2500 50  0000 C CNN
 F 1 "CONN_01X06" V 8450 2150 50  0000 C CNN
-F 2 "" H 8350 2150 60  0000 C CNN
+F 2 "JST-SH:JST-BM-06B-SRSS-TB" H 8350 2150 60  0001 C CNN
 F 3 "" H 8350 2150 60  0000 C CNN
 	1    8350 2150
@@
 	7750 2300 8150 2300
 $Comp
-L VPP #PWR5
+L VPP #PWR017
 U 1 1 5510A01A
 P 7850 1850
-F 0 "#PWR5" H 7850 1700 60  0001 C CNN
+F 0 "#PWR017" H 7850 1700 60  0001 C CNN
 F 1 "VPP" H 7850 2000 60  0000 C CNN
 F 2 "" H 7850 1850 60  0000 C CNN
@@
 $EndComp
 $Comp
-L GND #PWR7
+L GND #PWR018
 U 1 1 5510A020
 P 8100 2450
-F 0 "#PWR7" H 8100 2200 60  0001 C CNN
+F 0 "#PWR018" H 8100 2200 60  0001 C CNN
 F 1 "GND" H 8100 2300 60  0000 C CNN
 F 2 "" H 8100 2450 60  0000 C CNN
@@
 F 0 "P3" H 8350 3400 50  0000 C CNN
 F 1 "CONN_01X06" V 8450 3050 50  0000 C CNN
-F 2 "" H 8350 3050 60  0000 C CNN
+F 2 "JST-SH:JST-BM-06B-SRSS-TB" H 8350 3050 60  0001 C CNN
 F 3 "" H 8350 3050 60  0000 C CNN
 	1    8350 3050
@@
 	7750 3200 8150 3200
 $Comp
-L VPP #PWR9
+L VPP #PWR019
 U 1 1 5510A038
 P 7850 2750
-F 0 "#PWR9" H 7850 2600 60  0001 C CNN
+F 0 "#PWR019" H 7850 2600 60  0001 C CNN
 F 1 "VPP" H 7850 2900 60  0000 C CNN
 F 2 "" H 7850 2750 60  0000 C CNN
@@
 $EndComp
 $Comp
-L GND #PWR12
+L GND #PWR020
 U 1 1 5510A03E
 P 8100 3350
-F 0 "#PWR12" H 8100 3100 60  0001 C CNN
+F 0 "#PWR020" H 8100 3100 60  0001 C CNN
 F 1 "GND" H 8100 3200 60  0000 C CNN
 F 2 "" H 8100 3350 60  0000 C CNN
@@
 F 0 "P4" H 8350 4300 50  0000 C CNN
 F 1 "CONN_01X06" V 8450 3950 50  0000 C CNN
-F 2 "" H 8350 3950 60  0000 C CNN
+F 2 "JST-SH:JST-BM-06B-SRSS-TB" H 8350 3950 60  0001 C CNN
 F 3 "" H 8350 3950 60  0000 C CNN
 	1    8350 3950
@@
 	7750 4100 8150 4100
 $Comp
-L VPP #PWR15
+L VPP #PWR021
 U 1 1 5510A056
 P 7850 3650
-F 0 "#PWR15" H 7850 3500 60  0001 C CNN
+F 0 "#PWR021" H 7850 3500 60  0001 C CNN
 F 1 "VPP" H 7850 3800 60  0000 C CNN
 F 2 "" H 7850 3650 60  0000 C CNN
@@
 $EndComp
 $Comp
-L GND #PWR17
+L GND #PWR022
 U 1 1 5510A05C
 P 8100 4250
-F 0 "#PWR17" H 8100 4000 60  0001 C CNN
+F 0 "#PWR022" H 8100 4000 60  0001 C CNN
 F 1 "GND" H 8100 4100 60  0000 C CNN
 F 2 "" H 8100 4250 60  0000 C CNN
@@
 F 0 "P5" H 8350 5200 50  0000 C CNN
 F 1 "CONN_01X06" V 8450 4850 50  0000 C CNN
-F 2 "" H 8350 4850 60  0000 C CNN
+F 2 "JST-SH:JST-BM-06B-SRSS-TB" H 8350 4850 60  0001 C CNN
 F 3 "" H 8350 4850 60  0000 C CNN
 	1    8350 4850
@@
 	7750 5000 8150 5000
 $Comp
-L VPP #PWR19
+L VPP #PWR023
 U 1 1 5510A074
 P 7850 4550
-F 0 "#PWR19" H 7850 4400 60  0001 C CNN
+F 0 "#PWR023" H 7850 4400 60  0001 C CNN
 F 1 "VPP" H 7850 4700 60  0000 C CNN
 F 2 "" H 7850 4550 60  0000 C CNN
@@
 $EndComp
 $Comp
-L GND #PWR21
+L GND #PWR024
 U 1 1 5510A07A
 P 8100 5150
-F 0 "#PWR21" H 8100 4900 60  0001 C CNN
+F 0 "#PWR024" H 8100 4900 60  0001 C CNN
 F 1 "GND" H 8100 5000 60  0000 C CNN
 F 2 "" H 8100 5150 60  0000 C CNN
@@
 F 0 "P6" H 8350 6100 50  0000 C CNN
 F 1 "CONN_01X06" V 8450 5750 50  0000 C CNN
-F 2 "" H 8350 5750 60  0000 C CNN
+F 2 "JST-SH:JST-BM-06B-SRSS-TB" H 8350 5750 60  0001 C CNN
 F 3 "" H 8350 5750 60  0000 C CNN
 	1    8350 5750
@@
 	7750 5900 8150 5900
 $Comp
-L VPP #PWR23
+L VPP #PWR025
 U 1 1 5510A092
 P 7850 5450
-F 0 "#PWR23" H 7850 5300 60  0001 C CNN
+F 0 "#PWR025" H 7850 5300 60  0001 C CNN
 F 1 "VPP" H 7850 5600 60  0000 C CNN
 F 2 "" H 7850 5450 60  0000 C CNN
@@
 $EndComp
 $Comp
-L GND #PWR25
+L GND #PWR026
 U 1 1 5510A098
 P 8100 6050
-F 0 "#PWR25" H 8100 5800 60  0001 C CNN
+F 0 "#PWR026" H 8100 5800 60  0001 C CNN
 F 1 "GND" H 8100 5900 60  0000 C CNN
 F 2 "" H 8100 6050 60  0000 C CNN
