File: Schematics/panelized.kicad_pcb (KiCad board)
At the start: 2 copper layers, 84 x 50 mm, 154 parts, among them CON1 USB-MICRO-B, CON2 BARREL_JACK, IC1 ATXMEGA256A3BU-A, J1 AVR_JTAG_Header, P1 CONN_01X04, P1 CONN_01X06, P10 CONN_01X06, P11 CONN_01X06, P12 CONN_01X06, P13 CONN_01X02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

Commit message: sTUFF
Parts:
- removed the C1 at (193.5, 76.0) (x2)
- removed the C101 at (196.3, 78.7) (x2)
- removed the P1 at (204.9, 77.0) (x2)
- removed the P2 at (204.9, 69.0) (x2)
- removed the P3 at (198.5, 63.2) (x2)
- removed the P4 at (192.2, 69.0) (x2)
- removed the P5 at (192.2, 77.0) (x2)
- removed the P6 at (198.5, 82.8) (x2)
- removed the R1 at (196.2, 78.3) (x2)
- removed the R10 at (198.6, 75.0) (x2)
- removed the R11 at (197.0, 75.0) (x2)
- removed the R2 at (197.8, 78.3) (x2)
- removed the R3 at (199.4, 78.3) (x2)
- removed the R4 at (201.1, 78.3) (x2)
- removed the R5 at (196.2, 79.8) (x2)
- removed the R6 at (197.8, 79.8) (x2)
- removed the R7 at (199.4, 79.8) (x2)
- removed the R8 at (201.1, 79.8) (x2)
- removed the R9 at (200.2, 75.0) (x2)
- removed the U1 at (198.6, 71.8) (x2)
- added C1 (x2): C, Capacitors_SMD:C_0603, F.Cu at (193.5, 76.0)
- added C101 (x2): C, Capacitors_SMD:C_0603, B.Cu at (196.3, 78.7)
- added P1 (x2): CONN_01X04, JST-SH:JST-BM-04B-SRSS-TB, B.Cu at (204.9, 77.0)
- added P2 (x2): CONN_01X04, JST-SH:JST-BM-04B-SRSS-TB, B.Cu at (204.9, 69.0)
- added P3 (x2): CONN_01X04, JST-SH:JST-BM-04B-SRSS-TB, B.Cu at (198.5, 63.2)
- added P4 (x2): CONN_01X04, JST-SH:JST-BM-04B-SRSS-TB, B.Cu at (192.2, 69.0)
- added P5 (x2): CONN_01X04, JST-SH:JST-BM-04B-SRSS-TB, B.Cu at (192.2, 77.0)
- added P6 (x2): CONN_01X06, JST-SH:JST-BM-06B-SRSS-TB, B.Cu at (198.5, 82.8)
- added R1 (x2): 0R, Resistors_SMD:R_0603, F.Cu at (196.2, 78.3)
- added R10 (x2): 10k, Resistors_SMD:R_0603, B.Cu at (198.6, 75.0)
- added R11 (x2): 10k, Resistors_SMD:R_0603, B.Cu at (197.0, 75.0)
- added R2 (x2): 0R, Resistors_SMD:R_0603, F.Cu at (197.8, 78.3)
- added R3 (x2): 0R, Resistors_SMD:R_0603, F.Cu at (199.4, 78.3)
- added R4 (x2): 0R, Resistors_SMD:R_0603, F.Cu at (201.1, 78.3)
- added R5 (x2): 0R, Resistors_SMD:R_0603, F.Cu at (196.2, 79.8)
- added R6 (x2): 0R, Resistors_SMD:R_0603, F.Cu at (197.8, 79.8)
- added R7 (x2): 0R, Resistors_SMD:R_0603, F.Cu at (199.4, 79.8)
- added R8 (x2): 0R, Resistors_SMD:R_0603, F.Cu at (201.1, 79.8)
- added R9 (x2): 10k, Resistors_SMD:R_0603, B.Cu at (200.2, 75.0)
- added U1 (x2): PCA9685, Housings_SSOP:TSSOP-28_4.4x9.7mm_Pitch0.65mm, F.Cu at (198.6, 71.8)
Changed lines of the file:
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@@
       (psnegative false)
       (psa4output false)
-      (plotreference false)
-      (plotvalue true)
+      (plotreference true)
+      (plotvalue false)
       (plotinvisibletext false)
       (padsonsilk false)
